File: SmartFridgeProject.kicad_pcb (KiCad board)
At the start: 2 copper layers, 96.5 x 63.5 mm, 27 parts, among them J1 I2C_LCD_HEADER, J2 WIRELESS_UART, Q1 2N3904, SW2 threshold/set, SW3 mode/display, SW4 door_reed1, U1 ATmega328P-A, U2 AMS1117-3.3, U3 SHT31-DIS

Commit message: pcb trace finished; other misc. changes
Parts:
- removed SW4: door_reed1, Connector_PinHeader_2.54mm:PinHeader_1x02_P2.54mm_Vertical
- added door_reed1: MK24-B, Connector_PinHeader_2.54mm:PinHeader_1x02_P2.54mm_Vertical, F.Cu at (98.0, 88.5)
- moved R8 31.6 mm to (139.0, 105.0), turned to 90 degrees
- moved J2 27.5 mm to (134.0, 81.5)
- moved R10 25.5 mm to (127.0, 81.0), turned to 180 degrees
- moved Thermistor1 24.9 mm to (133.5, 127.0)
- moved C1 24.8 mm to (113.5, 104.0)
- moved R9 24.8 mm to (128.5, 85.0)
- moved R1 24.4 mm to (133.5, 115.5)
- moved U3 21.1 mm to (134.0, 102.0)
- moved BZ1 3.50 mm to (72.4, 120.0)
- moved C4 3.40 mm to (120.0, 95.2)
- moved J1 2.87 mm to (149.0, 92.5)
- moved R4 2.63 mm to (99.5, 102.6)
Routing:
- net /3.3V: track 0.00 -> 155.3 mm, vias 0 -> 8
- net GND: track 0.00 -> 67.7 mm, vias 0 -> 16
- net /SDA: track 0.00 -> 60.1 mm, vias 0 -> 2
- net /SCL: track 0.00 -> 58.0 mm, vias 0 -> 6
- net /INT0: track 0.00 -> 46.1 mm, vias 0 -> 4
- net /TEMP_ADC: track 0.00 -> 43.5 mm
- net /INT1: track 13.4 -> 56.0 mm, vias 0 -> 4
- net +5V: track 0.00 -> 39.3 mm
- net /RX: track 0.00 -> 26.8 mm, vias 0 -> 4
- net /TX: track 0.00 -> 26.5 mm, vias 0 -> 2
- net Net-(U1-PB1): track 0.00 -> 22.3 mm
- net Net-(U1-PD5): track 0.00 -> 16.3 mm, vias 0 -> 2
- net Net-(U1-PD4): track 0.00 -> 15.0 mm
- net Net-(U1-PD6): track 0.00 -> 13.6 mm, vias 0 -> 2
- net Net-(BZ1--): track 0.00 -> 12.5 mm
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- added copper zone on B.Cu, net GND
